Commit message: Added gazebo_ros2_control interface and rqt_joint_trajectory_controller

File: description/ic2d.xacro (robot description, xacro)
@@ -1,4 +1,7 @@
 <?xml version="1.0"?>
-<robot xmlns:xacro="http://www.ros.org/wiki/xacro"  name="IC2D">
+<robot xmlns:xacro="http://www.ros.org/wiki/xacro" name="IC2D">
+    <!-- Definitons -->
+    <xacro:property name="slider_upper" value="1.0" />
+    <xacro:property name="slider_lower" value="-1.0" />
     <!-- Useful Macros -->
     <xacro:macro name="include_geometry_file" params="filename">
@@ -17,7 +20,14 @@
     </xacro:macro>
     <!-- Specify some colours -->
+    <!-- Rviz color -->
     <material name="nickel">
         <color rgba="${193/255} ${183/255} ${131/255} 1"/>
     </material>
+    <!-- Gazebo color -->
+    <gazebo reference="base_link">
+        <material>
+            Gazebo/White
+        </material>
+    </gazebo>
     <!-- This first link called "world" is empty -->
     <link name="world"></link>
@@ -27,5 +37,5 @@
         <child link="base_link"/>
         <axis xyz="1 0 0"/>
-        <limit lower="${-pi/2}" upper="${pi/2}" velocity="340" effort="5000"/>
+        <limit lower="${slider_lower}" upper="${slider_upper}" velocity="340" effort="5000"/>
     </joint>
     <link name="base_link">
@@ -50,5 +60,5 @@
         <xacro:inertial_box mass="${base_global_mass}" dx="${base_global_width}"
                             dy="${base_global_height}" dz="${base_global_length}">
-                                <xacro:insert_block name="link_origin" />
+            <xacro:insert_block name="link_origin" />
         </xacro:inertial_box>
     </link>
@@ -56,11 +66,10 @@
     <!-- This plugin will publish the joint_states for the selected joints
             (which robot_state_publisher can then use to broadcast the approprate tf). -->
-    <gazebo>
-        <plugin name="gazebo_ros_joint_state_publisher"
-            filename="libgazebo_ros_joint_state_publisher.so">
+    <!-- gazebo>
+        <plugin name="gazebo_ros_joint_state_publisher" filename="libgazebo_ros_joint_state_publisher.so">
             <update_rate>20</update_rate>
             <joint_name>slider_joint</joint_name>
         </plugin>
-    </gazebo>
+    </gazebo -->
     <!-- This plugin will read a JointTrajectory message from the /set_joint_trajectory topic
             and move the machine accordingly. It's a bit clunky but it works. -->
@@ -69,8 +78,30 @@
     <!-- Here's an example message to publish to test it:
             ros2 topic pub -1 /set_joint_trajectory trajectory_msgs/msg/JointTrajectory  '{header: {frame_id: world}, joint_names: [slider_joint, arm_joint], points: [  {positions: {0.8,0.6}} ]}' -->
+    <!-- gazebo>
+        <plugin name="gazebo_ros_joint_pose_trajectory" filename="libgazebo_ros_joint_pose_trajectory.so">
+            <update_rate>2</update_rate>
+        </plugin>
+    </gazebo -->
+    <ros2_control name="GazeboSystem" type="system">
+        <hardware>
+            <plugin>gazebo_ros2_control/GazeboSystem</plugin>
+        </hardware>
+        <joint name="slider_joint">
+            <command_interface name="position">
+                <param name="min">-1.0</param>
+                <param name="max">1.0</param>
+            </command_interface>
+            <state_interface name="position">
+                <param name="initial_value">0.0</param>
+            </state_interface>
+            <state_interface name="velocity" />
+            <state_interface name="effort" />
+        </joint>
+    </ros2_control>
     <gazebo>
-        <plugin name="gazebo_ros_joint_pose_trajectory"
-            filename="libgazebo_ros_joint_pose_trajectory.so">
-            <update_rate>2</update_rate>
+        <plugin filename="libgazebo_ros2_control.so" name="gazebo_ros2_control">
+            <robot_param_node>robot_state_publisher</robot_param_node>
+            <robot_param>robot_description</robot_param>
+            <parameters>$(find ic2d_urdf)/config/ic2d_controllers.yaml</parameters>
         </plugin>
     </gazebo>

Commit message: Added effort_controller, it works but sim integration looks bad

File: description/ic2d.xacro (robot description, xacro)
@@ -2,6 +2,6 @@
 <robot xmlns:xacro="http://www.ros.org/wiki/xacro" name="IC2D">
     <!-- Definitons -->
-    <xacro:property name="slider_upper" value="1.0" />
-    <xacro:property name="slider_lower" value="-1.0" />
+    <xacro:property name="slider_upper" value="10.0" />
+    <xacro:property name="slider_lower" value="-10.0" />
     <!-- Useful Macros -->
     <xacro:macro name="include_geometry_file" params="filename">
@@ -63,24 +63,5 @@
         </xacro:inertial_box>
     </link>
-    <!-- Gazebo requires the use of plugins to interact with other systems such as ROS. -->
-    <!-- This plugin will publish the joint_states for the selected joints
-            (which robot_state_publisher can then use to broadcast the approprate tf). -->
-    <!-- gazebo>
-        <plugin name="gazebo_ros_joint_state_publisher" filename="libgazebo_ros_joint_state_publisher.so">
-            <update_rate>20</update_rate>
-            <joint_name>slider_joint</joint_name>
-        </plugin>
-    </gazebo -->
-    <!-- This plugin will read a JointTrajectory message from the /set_joint_trajectory topic
-            and move the machine accordingly. It's a bit clunky but it works. -->
-    <!-- You'll probably want to add damping to the joints to stop them it flopping around.
-            e.g. <dynamics damping="10.0" friction="10.0"/> -->
-    <!-- Here's an example message to publish to test it:
-            ros2 topic pub -1 /set_joint_trajectory trajectory_msgs/msg/JointTrajectory  '{header: {frame_id: world}, joint_names: [slider_joint, arm_joint], points: [  {positions: {0.8,0.6}} ]}' -->
-    <!-- gazebo>
-        <plugin name="gazebo_ros_joint_pose_trajectory" filename="libgazebo_ros_joint_pose_trajectory.so">
-            <update_rate>2</update_rate>
-        </plugin>
-    </gazebo -->
+    <!-- Necessary config/tags for ros2_control interface with Gazebo Classic -->
     <ros2_control name="GazeboSystem" type="system">
         <hardware>
@@ -88,7 +69,7 @@
         </hardware>
         <joint name="slider_joint">
-            <command_interface name="position">
-                <param name="min">-1.0</param>
-                <param name="max">1.0</param>
+            <command_interface name="effort">
+                <param name="min">-10000.0</param>
+                <param name="max">10000.0</param>
             </command_interface>
             <state_interface name="position">

Commit message: Added Gazebo world file and setup joint dynamics

File: description/ic2d.xacro (robot description, xacro)
@@ -4,4 +4,6 @@
     <xacro:property name="slider_upper" value="10.0" />
     <xacro:property name="slider_lower" value="-10.0" />
+    <xacro:property name="slider_effort_lim" value="10000" />
+    <xacro:property name="slider_damping" value="1.00" />
     <!-- Useful Macros -->
     <xacro:macro name="include_geometry_file" params="filename">
@@ -27,6 +29,11 @@
     <gazebo reference="base_link">
         <material>
-            Gazebo/White
+            Gazebo/Gold
         </material>
+    </gazebo>
+    <!-- Gazebo Joint Dynamics -->
+    <gazebo reference="slider_joint">
+        <springStiffness>1000</springStiffness>
+        <springReference>0</springReference>
     </gazebo>
     <!-- This first link called "world" is empty -->
@@ -37,5 +44,12 @@
         <child link="base_link"/>
         <axis xyz="1 0 0"/>
-        <limit lower="${slider_lower}" upper="${slider_upper}" velocity="340" effort="5000"/>
+        <!-- calibration: the reference positions of the joint,
+        used to calibrate the absolute position of the joint. -->
+        <!-- calibration rising="0.0" /-->
+        <!-- dynamics: an element specifying physical properties of the joint.
+        These values are used to specify modeling properties of the joint,
+        particularly useful for simulation.-->
+        <dynamics damping="${slider_damping}" friction="0.0" />
+        <limit lower="${slider_lower}" upper="${slider_upper}" velocity="340" effort="${slider_effort_lim}"/>
     </joint>
     <link name="base_link">
@@ -50,5 +64,5 @@
             <origin xyz="${-base_global_width/2} ${base_global_length/2} 0" rpy="${pi/2} 0 0" />
             <xacro:include_geometry_file filename="base_global"/>
-            <material name="nickel" />
+            <material name="nickel" /> <!-- for Rviz   -->
         </visual>
         <collision>
@@ -76,6 +90,10 @@
                 <param name="initial_value">0.0</param>
             </state_interface>
-            <state_interface name="velocity" />
-            <state_interface name="effort" />
+            <state_interface name="velocity">
+                <param name="initial_value">0.0</param>
+            </state_interface>
+            <state_interface name="effort">
+                <param name="initial_value">0.0</param>
+            </state_interface>
         </joint>
     </ros2_control>

Commit message: Fix rviz2 STL loading failure

File: description/ic2d.xacro (robot description, xacro)
@@ -9,5 +9,5 @@
     <xacro:macro name="include_geometry_file" params="filename">
         <geometry>
-            <mesh filename="$(find ic2d_urdf)/meshes/${filename}.STL" scale="0.001 0.001 0.001"/>
+            <mesh filename="file://$(find ic2d_urdf)/meshes/${filename}.STL"/>
         </geometry>
     </xacro:macro>

File: description/ic2d_position.xacro (robot description, xacro)
@@ -9,5 +9,5 @@
     <xacro:macro name="include_geometry_file" params="filename">
         <geometry>
-            <mesh filename="$(find ic2d_urdf)/meshes/${filename}.STL"/>
+            <mesh filename="file://$(find ic2d_urdf)/meshes/${filename}.STL"/>
         </geometry>
     </xacro:macro>
